File: hardware/black_scope/black_scope.kicad_sch (KiCad schematic)
At the start: 72 parts, among them J1 Conn_ARM_JTAG_SWD_10, J3 Conn_01x02, J4 Conn_02x04_Odd_Even, J5 Conn_02x02_Odd_Even, P1 USB_C_Plug_USB2.0, Q1 S8050, SW1 SW_Push, SW2 SW_Push, U1 MCP73831-2-OT, U2 XC6206PxxxMR, U3 STM32G473VE, U4 LMV358, U5 XPT2046TS, U6 TFT035IPS, U7 QSPI_PSRAM, U8 LMV324, Y1 Crystal_GND24

Commit message: - Added images
Parts:
- C1, C10, C11, C12, C13, C14, C15, C16, C17, C18, C19, C20, C21, C5, C9: value C -> 100n
- C2, C3: value C -> 10p
- C4, C6, C7, C8: value C -> 270n
- L1, L2: value L -> 47u
- R1, R19: value R -> 22
- R10, R9: value R -> 51
- R2, R23, R24, R26: value R -> 10k
- R20, R21: value R -> 12
- R22, R4: value R -> 1k
- R3: value R -> 6.8k
Other:
- note added: "! Change boot polarity ! Add pull-down to DAC2-OUT1 - Add holes for TFT - Chnage charging led - Move battery connector - Add digital channels? - Add battery measurement - Move JTAG connector - Add resistor and capacitor values - bigger diodes footprint"

Commit message: - Update fw
Other:
- note added: "- Fix ADC noise issues."
- note added: "- Fix TFT connector location - Fix BJT pintout - Fit BL resistor values. 50Ohm - Change OPAMP ADC and DAC IC with bigger BW - Add capacitors to ADC channels"

Commit message: - Fix PCB issues - Add datasheets
Parts:
- removed Q1: S8050, Package_TO_SOT_SMD:SOT-23, symbol Transistor_BJT:S8050
- added C22: 100n, Capacitor_SMD:C_0603_1608Metric_Pad1.08x0.95mm_HandSolder, symbol Device:C
- added C23, C24, C25, C26: 100p, Capacitor_SMD:C_0603_1608Metric_Pad1.08x0.95mm_HandSolder, symbol Device:C
- added D4: D_Schottky_Dual_CommonCathode_AAK_Parallel, symbol Device:D_Schottky_Dual_CommonCathode_AAK_Parallel
- added Q3: Q_NPN_BEC, Package_TO_SOT_SMD:SOT-23, symbol Device:Q_NPN_BEC
- added R25: 10k, Resistor_SMD:R_0603_1608Metric_Pad0.98x0.95mm_HandSolder, symbol Device:R
- D1, D3: footprint Diode_SMD:D_0603_1608Metric_Pad1.05x0.95mm_HandSolder -> Diode_SMD:D_1206_3216Metric_Pad1.42x1.75mm_HandSolder
- R11, R13, R15, R17: value R -> 2k7
- R12, R14, R16, R18: value R -> 4k3
- R20, R21: value 12 -> 51
- R5, R6, R7, R8: value R -> 8k2
Connections:
- net +3.3V: now also SW2.2, U6.8 (IM1); no longer U6.7 (IM0)
- net BOOT0: now also SW2.1
- net DAC2_OUT1: now also C22.1, R25.2
- net GND: now also R2.1, U6.7 (IM0), C22.2, C23.2, C24.2, C25.2, C26.2, Q3.2 (E), R25.1; no longer D2.1 (K), SW2.1, U6.8 (IM1)
- net VBUS: now also D2.2 (A)
- net at R4.1: now also U1.1 (STAT); no longer D2.2 (A)
- net at R11.1, R12.2, R5.2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: now also C23.1
- net at R22.1: now also Q3.1 (B)
- net at R17.1, R18.2, R8.2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: now also C26.1
- net at R15.1, R16.2, R7.2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: now also C25.1
- net at R20.2, R21.2: now also Q3.3 (C)
- net at R13.1, R14.2, R6.2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: now also C24.1
- net at R4.2: now also D2.1 (K); no longer U1.1 (STAT)
Other:
- note added: "+ Change boot polarity + Add pull-down to DAC2-OUT1 + Add capacitor to DAC2-OUT1 + Add holes for TFT + Chnage charging led - Move battery connector - Add digital channels? - Add battery measurement - Move JTAG connector + Add resistor and capacitor values + bigger diodes footprint"
- note added: "+ Fix TFT connector location + Fix TFT IMO selection + Fix BJT pintout + Fit BL resistor values. 50Ohm - Change OPAMP ADC and DAC IC with bigger BW + Add capacitors to ADC channels - Change schottky diodes to SOT23-3"
- note added: "0.5% tolerance"
- note added: "IM[2:0] Interface Data Pin in Use 010 16-bit bus DB15:0"
- note removed: "! Change boot polarity ! Add pull-down to DAC2-OUT1 - Add holes for TFT - Chnage charging led - Move battery connector - Add digital channels? - Add battery measurement - Move JTAG connector - Add resistor and capacitor values - bigger diodes footprint"
- note removed: "- Fix TFT connector location - Fix BJT pintout - Fit BL resistor values. 50Ohm - Change OPAMP ADC and DAC IC with bigger BW - Add capacitors to ADC channels"
- note removed: "CHECK PINOUT"
- moved on the sheet: D2, J4, R11, R12, R13, R14, R15, R16, R17, R18, R2, R4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

Commit message: - Gerber files v2
Parts:
- added C27, C28, C29, C30: 100n, Capacitor_SMD:C_0603_1608Metric_Pad1.08x0.95mm_HandSolder, symbol Device:C
- added J2: Conn_02x06_Odd_Even, Connector_PinHeader_2.54mm:PinHeader_2x06_P2.54mm_Vertical_SMD, symbol Connector_Generic:Conn_02x06_Odd_Even
- D4: footprint (none) -> Package_TO_SOT_SMD:SOT-23
Connections:
- net GND: now also C27.2, C28.2, C29.2, C30.2
- net XN: now also C28.1
- net XP: now also C30.1
- net YN: now also C27.1
- net YP: now also C29.1
Other:
- note added: "+ Change boot polarity + Add pull-down to DAC2-OUT1 + Add capacitor to DAC2-OUT1 + Add holes for TFT + Chnage charging led + Move battery connector - Add digital channels? - Add battery measurement - Move JTAG connector + Add resistor and capacitor values + bigger diodes footprint"
- note added: "+ Fix TFT connector location + Fix TFT IMO selection + Fix BJT pintout + Fit BL resistor values. 50Ohm + Change OPAMP ADC and DAC IC with bigger BW + Add capacitors to ADC channels - Change schottky diodes to SOT23-3"
- note added: "595-OPA2322AIDGKR"
- note added: "595-OPA4322AIPWR"
- note added: "SMD connector 200-TSM10302LDH"
- note removed: "+ Change boot polarity + Add pull-down to DAC2-OUT1 + Add capacitor to DAC2-OUT1 + Add holes for TFT + Chnage charging led - Move battery connector - Add digital channels? - Add battery measurement - Move JTAG connector + Add resistor and capacitor values + bigger diodes footprint"
- note removed: "+ Fix TFT connector location + Fix TFT IMO selection + Fix BJT pintout + Fit BL resistor values. 50Ohm - Change OPAMP ADC and DAC IC with bigger BW + Add capacitors to ADC channels - Change schottky diodes to SOT23-3"

Commit message: - Improve FPS
Other:
- note added: "595-OPA2322AIDGKR or 595-OPA2834IDGKR"
- note added: "Thick Film Resistors 0.5% 10K Input impedance 667-ERJ-3RBD2701V 667-ERJ-3RBD4301V 667-ERJ-3RBD8201V Thick Film Resistors 0.5%. 100K Input impedance 667-ERJ-3RBD2702V 667-ERJ-3RBD8202V 667-ERJ-3RBD4302V"
- note removed: "595-OPA2322AIDGKR"
Changed lines of the file:
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@@
     (effects (font (size 3 3) (thickness 0.6) bold italic) (justify left bottom))
   )
-  (text "SMD connector\n200-TSM10302LDH" (at 402.59 38.1 0)
+  (text "SMD connector\n200-TSM10302LDH" (at 21.59 288.29 0)
     (effects (font (size 3 3)) (justify left bottom))
   )
@@
     (at 414.02 96.52 0)
     (effects (font (size 3 3)) (justify left bottom))
+  )
+  (text "Thick Film Resistors 0.5%\n10K Input impedance\n667-ERJ-3RBD2701V\n667-ERJ-3RBD4301V\n667-ERJ-3RBD8201V\n\nThick Film Resistors 0.5%.\n100K Input impedance\n667-ERJ-3RBD2702V\n667-ERJ-3RBD8202V\n667-ERJ-3RBD4302V"
+    (at 85.09 275.59 0)
+    (effects (font (size 1.27 1.27)) (justify left bottom))
   )
   (text "CPU MISC" (at 190.5 142.24 0)
@@
     (effects (font (size 3 3) (thickness 0.6) bold italic) (justify left bottom))
   )
-  (text "595-OPA2322AIDGKR" (at 123.19 270.51 0)
+  (text "595-OPA2322AIDGKR\nor\n595-OPA2834IDGKR" (at 123.19 275.59 0)
     (effects (font (size 1.27 1.27)) (justify left bottom))
   )

Commit message: - Reduce buffers len to 512 and also timers one pulse values. - Move nuklear context as a global scope so it dont need to be in the freertos heap - FreeRTOS config, change configTOTAL_HEAP_SIZE from 32k to 8k Refactor wavegen Add ui functionality to control wavegen - Add enable clip/scissor in nuklear glue - Change defaultTask_attributes stack size from 16k to 2k - Increase FPS to 20 to 40 (CPU limits to 25 when UI is rendering) - Reduce the timeout for auto trigger mode.
Parts:
- R20, R21: value 51 -> 27
Other:
- note added: "+ Change BL resistors to 27Ohm - Add schotty diodes in parallel"
Changed lines of the file:
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@@
     (effects (font (size 3 3)) (justify left bottom))
   )
+  (text "+ Change BL resistors to 27Ohm\n- Add schotty diodes in parallel"
+    (at 368.3 33.02 0)
+    (effects (font (size 2 2)) (justify left bottom))
+  )
   (text "Thick Film Resistors 0.5%\n10K Input impedance\n667-ERJ-3RBD2701V\n667-ERJ-3RBD4301V\n667-ERJ-3RBD8201V\n\nThick Film Resistors 0.5%.\n100K Input impedance\n667-ERJ-3RBD2702V\n667-ERJ-3RBD8202V\n667-ERJ-3RBD4302V"
     (at 85.09 275.59 0)
@@
       (effects (font (size 1.27 1.27)))
     )
-    (property "Value" "51" (at 455.93 228.6 90)
+    (property "Value" "27" (at 455.93 228.6 90)
       (effects (font (size 1.27 1.27)))
     )
@@
       (effects (font (size 1.27 1.27)))
     )
-    (property "Value" "51" (at 455.93 238.76 90)
+    (property "Value" "27" (at 455.93 238.76 90)
       (effects (font (size 1.27 1.27)))
     )

Commit message: Long time update
Parts:
- added C31, C32: 270n, Capacitor_SMD:C_0603_1608Metric_Pad1.08x0.95mm_HandSolder, symbol Device:C
- added L3: 47u, Inductor_SMD:L_0603_1608Metric_Pad1.05x0.95mm_HandSolder, symbol Device:L
- added R27, R28, R29, R30: 27, Resistor_SMD:R_0603_1608Metric_Pad0.98x0.95mm_HandSolder, symbol Device:R
- added TP5, TP6: TestPoint, TestPoint:TestPoint_Pad_D1.0mm, symbol Connector:TestPoint
- added U9: XC6206PxxxMR, Package_TO_SOT_SMD:SOT-23-3, symbol Regulator_Linear:XC6206PxxxMR
- D1, D3: Mouser REF (none) -> 512-SS24FL
- D4: Mouser REF (none) -> 750-BAT54C-HF
- J1: Mouser REF (none) -> 649-221121-00010T4LF
- J2: Mouser REF (none) -> 200-TSM10302LDH
- L1, L2: Mouser REF (none) -> 80-L0603B470KPWFT
- P1: Mouser REF (none) -> 640-USB4105-GF-A
- Q3: Mouser REF (none) -> 750-SS8050-G
- R11, R13, R15, R17: Mouser REF (none) -> 667-ERJ-3RBD2701V
- R12, R14, R16, R18: Mouser REF (none) -> 667-ERJ-3RBD4301V
- R5, R6, R7, R8: Mouser REF (none) -> 667-ERJ-3RBD8201V
- SW1, SW2: Mouser REF (none) -> 688-SKRKAHE010
- U1: Mouser REF (none) -> 579-MCP73831T-2DCIOT
- U2: Mouser REF (none) -> 579-MCP1700T3302E/TT
- U3: Mouser REF (none) -> 511-STM32G473VET6
- U4: Mouser REF (none) -> 595-LMV358IDR
- U5: Mouser REF (none) -> 595-TSC2046EIPWR
- U6: Mouser REF (none) -> 649-62684-50210E9ALF
- U7: Mouser REF (none) -> 878-APS6404L-3SQR-SN
- U8: Mouser REF (none) -> 595-OPA4322AIPWR
- Y1: Mouser REF (none) -> 732-322524F20GAC0
Connections:
- net +3.3V: no longer L1.1
- net +3.3VA: now also TP5.1
- net GND: now also L3.1; no longer C13.2, C14.2, C16.2, C18.2, C22.2, C23.2, C24.2, C25.2, C26.2, C7.2, C8.2, J4.2 (Pin_2), J4.4 (Pin_4), J4.6 (Pin_6), J4.8 (Pin_8), J5.2 (Pin_2), J5.4 (Pin_4), R12.1, R14.1, R16.1, R18.1, R25.1, U3.35 (VSSA), U4.4 (V-), U8.11 (V-)
- net SPI3_MISO: now also R28.1; no longer U5.12 (DOUT)
- net SPI3_MOSI: now also R27.1; no longer U5.14 (DIN)
- net SPI3_NSS: now also R30.1; no longer R26.2, U5.15 (~{CS})
- net SPI3_SCLK: now also R29.1; no longer U5.16 (DCLK)
- net at C4.1, D1.1 (K), D3.1 (K)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: now also C31.1, U9.3 (VI)
- net GNDA: now reaches J2.10 (Pin_10)
- net GNDA: now also C13.2, C14.2, C16.2, C18.2, C22.2, C23.2, C24.2, C25.2, C26.2, C7.2, C8.2, J2.12 (Pin_12), J2.2 (Pin_2), J2.4 (Pin_4), J2.6 (Pin_6), J2.8 (Pin_8), J4.2 (Pin_2), J4.4 (Pin_4), J4.6 (Pin_6), J4.8 (Pin_8), J5.2 (Pin_2), J5.4 (Pin_4), R12.1, R14.1, R16.1, R18.1, R25.1, U3.35 (VSSA), U4.4 (V-), U8.11 (V-), C31.2, C32.2, L3.2, TP6.1, U9.1 (GND)
- new net: R29.2, U5.16 (DCLK)
- new net: C32.1, L1.1, U9.2 (VO)
- new net: R27.2, U5.14 (DIN)
- new net: R28.2, U5.12 (DOUT)
- new net: R26.2, R30.2, U5.15 (~{CS})
Other:
- moved on the sheet: D4, R26
